Commit message: 3d part on top

File: src/my_robot_description/urdf/rubot/rubot_mecanum_custom.urdf (robot description, URDF)
Before this commit: robot rubot, 9 links, 8 joints
Links:
- added link top_part, mass 0.08; collision box size=0.06 0.04 0.02; visual box size=0.06 0.04 0.02
Joints:
- added joint joint_top_part: type fixed, parent base_link, child top_part, origin xyz=0.0 0.0 0.13 rpy=0 0 0

Commit message: modified 3d part

File: src/my_robot_description/urdf/rubot/rubot_mecanum_custom.urdf (robot description, URDF)
Before this commit: robot rubot, 10 links, 9 joints
Links:
- added link arm_base, mass 0.05; collision cylinder length=0.1 radius=0.012; visual cylinder length=0.1 radius=0.012
- added link arm_upper, mass 0.05; collision cylinder length=0.1 radius=0.012; visual cylinder length=0.1 radius=0.012
- link top_part: geometry collision box size=0.05 0.05 0.009; visual box size=0.05 0.05 0.009
Joints:
- added joint joint_arm_base: type fixed, parent top_part, child arm_base, origin xyz=0 0 0.01 rpy=0 0 0
- added joint joint_arm_upper: type fixed, parent arm_base, child arm_upper, origin xyz=0 0 0.098 rpy=0 0 0
- joint joint_top_part: axis (none) -> 0 1 0; origin xyz=0.0 0.0 0.13 rpy=0 0 0 -> xyz=0.1 0.0 0.092 rpy=0 0 0
